File: hardware/VehicleAccessoryControllerTestBoard/VehicleAccessoryControllerTestBoard.kicad_pcb (KiCad board)
At the start: 4 copper layers, 55 x 41 mm, 52 parts, among them J501 Input, J502 Front Conn, J503 Rear Conn, J506 USB_Mini-B, Q201 BSS138, Q202 BSS138, SW301 ON/OFF, U103 TPS3710, U104 SI8710CC-B-IS, U105 CP2102N-A02-GQFN24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

Commit message: test board layout
Parts:
- removed D602: LED_ALT, VehicleAccessoryController:LED_0603
- removed R707: 430R, VehicleAccessoryController:R_0603
- removed REF**: GND_Stitch_Via, VehicleAccessoryController:GND_Stitch_Via
- added J507: Conn_01x02_Male, Connector_PinHeader_2.54mm:PinHeader_1x02_P2.54mm_Vertical, F.Cu at (126.0, 103.0)
- added J508: Conn_01x08_Male, Connector_PinHeader_2.54mm:PinHeader_1x08_P2.54mm_Vertical, F.Cu at (160.9, 80.0)
- moved fid1 9.49 mm to (126.0, 80.0)
- moved fid2 9.49 mm to (177.0, 80.0)
- moved fid3 9.00 mm to (177.0, 120.0)
- moved C811 7.70 mm to (147.7, 108.0), turned to 90 degrees
- moved C805 1.00 mm to (143.0, 84.0)
- moved D601 1.00 mm to (160.0, 85.0)
- moved R706 1.00 mm to (156.0, 85.0)
- moved C806 0.10 mm to (158.1, 103.0)
- moved C807 0.10 mm to (158.1, 105.0)
- moved C808 0.10 mm to (158.1, 107.0)
- moved C809 0.10 mm to (158.1, 109.0)
- moved R728 0.10 mm to (158.1, 97.5)
- moved R731 0.10 mm to (157.1, 100.0)
- moved R732 0.10 mm to (159.1, 100.0)
Routing:
- net /PARK_REAR: track 0.00 -> 39.1 mm, vias 0 -> 1
- net /328P_RXD: track 0.00 -> 31.3 mm, vias 0 -> 1
- net /328P_TXD: track 0.00 -> 28.7 mm, vias 0 -> 1
- net /SHIELD: track 0.00 -> 26.5 mm
- net /CTRL: track 0.00 -> 22.0 mm
- net VBUS: track 4.25 -> 25.3 mm, vias 0 -> 2
- net /D+: track 0.00 -> 18.3 mm, vias 0 -> 2
- net /PARK_FRONT: track 0.00 -> 16.1 mm, vias 0 -> 1
- net +5V: track 3.43 -> 19.2 mm, vias 0 -> 2
- net /D-: track 0.00 -> 14.9 mm, vias 0 -> 2
- net VDD: track 2.00 -> 15.5 mm, vias 0 -> 5
- net /ACC_IN: track 0.00 -> 11.2 mm
- net /ACC: track 0.00 -> 10.3 mm
- net /TX_LED: track 0.00 -> 9.45 mm
- net Net-(C811-Pad2): track 0.00 -> 7.70 mm
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- added copper zone on In1.Cu, net +12VA
- added copper zone on In1.Cu, net +5V
- added copper zone on In2.Cu, net GND
- added copper zone on B.Cu, net GNDA
- added copper zone on F.Cu, net GNDA
- added copper zone on In2.Cu, net GNDA
- added copper zone on B.Cu, net GNDD
- added copper zone on F.Cu, net GNDD
- added copper zone on In2.Cu, net GNDD
- added copper zone on In1.Cu, net VDD
- removed copper zone on In2.Cu, net +5V
Other:
- board size 55 x 41 mm -> 55 x 44 mm

Commit message: test board schematic/layout updates, gerbers
Parts:
- added TP1: TestPoint, TestPoint:TestPoint_Pad_1.0x1.0mm, F.Cu at (146.9, 109.5)
- moved C811 2.00 mm to (147.7, 106.0)
Connections:
- C806 pad 2: GND -> GNDD
- C807 pad 2: GND -> GNDD
- C808 pad 2: GND -> GNDD
- C809 pad 2: GND -> GNDD
Routing:
- net /328P_RESET: track 0.00 -> 2.83 mm
- net Net-(C811-Pad2): track 7.70 -> 5.70 mm
- net GNDD: track 5.82 -> 7.00 mm, vias 7 -> 12
- net GND: vias 8 -> 6
Other:
- board text added: "Designed by Ops V0.0"
- board text added: "Vehicle Accessory Controller Test Board"

Commit message: test board PDFs, label updates, merge duplicates on BOMs
Parts:
- R731: value 22.1k -> 22k1
- R732: value 47.5k -> 47k5
Changed lines of the file:
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@@
-(kicad_pcb (version 20171130) (host pcbnew 5.1.4-e60b266~84~ubuntu18.04.1)
+(kicad_pcb (version 20171130) (host pcbnew 5.1.5-52549c5~84~ubuntu18.04.1)
   (general
     (thickness 1.6)
@@
   (title_block
     (title "Vehicle Accessory Controller Test Board")
-    (date 2019-11-15)
+    (date 2019-11-22)
     (rev 0.0)
     (company Noctivore)
@@
   )
   (layers
-    (0 F.Cu signal)
+    (0 F.Cu signal hide)
     (1 In1.Cu power hide)
     (2 In2.Cu power hide)
-    (31 B.Cu signal)
-    (32 B.Adhes user)
-    (33 F.Adhes user)
+    (31 B.Cu signal hide)
+    (32 B.Adhes user hide)
+    (33 F.Adhes user hide)
     (34 B.Paste user)
     (35 F.Paste user)
@@
     (37 F.SilkS user)
     (38 B.Mask user hide)
-    (39 F.Mask user)
+    (39 F.Mask user hide)
     (40 Dwgs.User user)
     (41 Cmts.User user)
@@
     (47 F.CrtYd user)
     (48 B.Fab user)
-    (49 F.Fab user hide)
+    (49 F.Fab user)
   )
   (setup
@@
       (effects (font (size 0.5 0.5) (thickness 0.125)))
     )
-    (fp_text value 22.1k (at 0 2 90) (layer F.Fab)
+    (fp_text value 22k1 (at 0 2 90) (layer F.Fab)
       (effects (font (size 1 1) (thickness 0.15)))
     )
@@
       (effects (font (size 0.5 0.5) (thickness 0.125)))
     )
-    (fp_text value 47.5k (at 0 3 90) (layer F.Fab)
-      (effects (font (size 1 1) (thickness 0.15)))
-    )
+    (fp_text value 47k5 (at 0 3 90) (layer F.Fab)
+      (effects (font (size 1 1) (thickness 0.15)))
+    )
