File: hardware/VehicleAccessoryControllerTestBoard/VehicleAccessoryControllerTestBoard.sch (KiCad schematic (older format))
At the start: 51 parts, among them J501 Input, J502 Front Conn, J503 Rear Conn, J506 USB_Mini-B, Q201 BSS138, Q202 BSS138, SW301 ON/OFF, U103 TPS3710, U104 SI8710CC-B-IS, U105 CP2102N-A02-GQFN24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

Commit message: test board layout
Parts:
- removed D602: LED_ALT, VehicleAccessoryController:LED_0603, symbol Device:LED_ALT
- removed R707: 430R, VehicleAccessoryController:R_0603, symbol Device:R
- added J507: Conn_01x02_Male, Connector_PinHeader_2.54mm:PinHeader_1x02_P2.54mm_Vertical, symbol Connector:Conn_01x02_Male
- added J508: Conn_01x08_Male, Connector_PinHeader_2.54mm:PinHeader_1x08_P2.54mm_Vertical, symbol Connector:Conn_01x08_Male
Connections:
- net +5V: now also J508.1 (Pin_1)
- net 328P_RXD: now also J508.7 (Pin_7)
- net 328P_TXD: now also J508.6 (Pin_6)
- net ACC: now also J508.5 (Pin_5)
- net CTRL: now also J507.1 (Pin_1)
- net GND: now also J508.8 (Pin_8)
- net GNDA: now also J507.2 (Pin_2)
- net PARK_FRONT: now also J508.2 (Pin_2)
- net PARK_REAR: now also J508.3 (Pin_3)
- net PARK_STATUS: now also J508.4 (Pin_4)
Other:
- moved on the sheet: C811, C812, C813, D605, J506, R728, SW301, U105, U106

Commit message: test board schematic/layout updates, gerbers
Parts:
- added TP1: TestPoint, TestPoint:TestPoint_Pad_1.0x1.0mm, symbol Connector:TestPoint
Connections:
- net 328P_RESET: now also TP1.1
- net GND: no longer C806.2, C807.2, C808.2, C809.2
- net GNDD: now also C806.2, C807.2, C808.2, C809.2
Changed lines of the file:
@@
 Sheet 1 1
 Title "Vehicle Accessory Controller Test Board"
-Date "2019-11-14"
+Date "2019-11-15"
 Rev "0.0"
 Comp "Noctivore"
@@
 	1    0    0    -1
 $EndComp
-$Comp
-L power:GND #PWR0149
-U 1 1 5DC4B377
-P 4450 7275
-F 0 "#PWR0149" H 4450 7025 50  0001 C CNN
-F 1 "GND" H 4455 7102 50  0000 C CNN
-F 2 "" H 4450 7275 50  0001 C CNN
-F 3 "" H 4450 7275 50  0001 C CNN
-	1    4450 7275
-	1    0    0    -1
-$EndComp
-$Comp
-L power:GND #PWR0150
-U 1 1 5DC546B1
-P 4900 7275
-F 0 "#PWR0150" H 4900 7025 50  0001 C CNN
-F 1 "GND" H 4905 7102 50  0000 C CNN
-F 2 "" H 4900 7275 50  0001 C CNN
-F 3 "" H 4900 7275 50  0001 C CNN
-	1    4900 7275
-	1    0    0    -1
-$EndComp
 Wire Wire Line
 	4450 6825 4450 6900
@@
 F 3 "" H 5850 6825 50  0001 C CNN
 	1    5850 6825
-	1    0    0    -1
-$EndComp
-$Comp
-L power:GND #PWR0154
-U 1 1 5DCBD7D2
-P 5400 7275
-F 0 "#PWR0154" H 5400 7025 50  0001 C CNN
-F 1 "GND" H 5405 7102 50  0000 C CNN
-F 2 "" H 5400 7275 50  0001 C CNN
-F 3 "" H 5400 7275 50  0001 C CNN
-	1    5400 7275
-	1    0    0    -1
-$EndComp
-$Comp
-L power:GND #PWR0155
-U 1 1 5DCBD7D8
-P 5850 7275
-F 0 "#PWR0155" H 5850 7025 50  0001 C CNN
-F 1 "GND" H 5855 7102 50  0000 C CNN
-F 2 "" H 5850 7275 50  0001 C CNN
-F 3 "" H 5850 7275 50  0001 C CNN
-	1    5850 7275
 	1    0    0    -1
 $EndComp
@@
 Wire Wire Line
 	1475 2725 1325 2725
+$Comp
+L Connector:TestPoint TP1
+U 1 1 5DD0862F
+P 8950 6400
+F 0 "TP1" V 8875 6475 50  0000 L CNN
+F 1 "TestPoint" V 9025 6375 50  0000 L CNN
+F 2 "TestPoint:TestPoint_Pad_1.0x1.0mm" H 9150 6400 50  0001 C CNN
+F 3 "~" H 9150 6400 50  0001 C CNN
+	1    8950 6400
+	0    1    1    0
+$EndComp
+Text Label 8800 6400 2    50   ~ 0
+328P_RESET
+Wire Wire Line
+	8800 6400 8950 6400
+$Comp
+L power:GNDD #PWR?
+U 1 1 5DD412B8
+P 4450 7275
+F 0 "#PWR?" H 4450 7025 50  0001 C CNN
+F 1 "GNDD" H 4454 7120 50  0000 C CNN
+F 2 "" H 4450 7275 50  0001 C CNN
+F 3 "" H 4450 7275 50  0001 C CNN
+	1    4450 7275
+	1    0    0    -1
+$EndComp
+$Comp
+L power:GNDD #PWR?
+U 1 1 5DD434DA
+P 4900 7275
+F 0 "#PWR?" H 4900 7025 50  0001 C CNN
+F 1 "GNDD" H 4904 7120 50  0000 C CNN
+F 2 "" H 4900 7275 50  0001 C CNN
+F 3 "" H 4900 7275 50  0001 C CNN
+	1    4900 7275
+	1    0    0    -1
+$EndComp
+$Comp
+L power:GNDD #PWR?
+U 1 1 5DD437E8
+P 5400 7275
+F 0 "#PWR?" H 5400 7025 50  0001 C CNN
+F 1 "GNDD" H 5404 7120 50  0000 C CNN
+F 2 "" H 5400 7275 50  0001 C CNN
+F 3 "" H 5400 7275 50  0001 C CNN
+	1    5400 7275
+	1    0    0    -1
+$EndComp
+$Comp
+L power:GNDD #PWR?
+U 1 1 5DD43A92
+P 5850 7275
+F 0 "#PWR?" H 5850 7025 50  0001 C CNN
+F 1 "GNDD" H 5854 7120 50  0000 C CNN
+F 2 "" H 5850 7275 50  0001 C CNN
+F 3 "" H 5850 7275 50  0001 C CNN
+	1    5850 7275
+	1    0    0    -1
+$EndComp
 $EndSCHEMATC

Commit message: test board PDFs, label updates, merge duplicates on BOMs
Parts:
- R731: value 22.1k -> 22k1
- R732: value 47.5k -> 47k5
Changed lines of the file:
@@
 EESchema Schematic File Version 4
-LIBS:VehicleAccessoryControllerTestBoard-cache
 EELAYER 30 0
 EELAYER END
@@
 Sheet 1 1
 Title "Vehicle Accessory Controller Test Board"
-Date "2019-11-15"
+Date "2019-11-22"
 Rev "0.0"
 Comp "Noctivore"
@@
 P 3900 5450
 F 0 "R732" H 3975 5400 50  0000 L CNN
-F 1 "47.5k" H 3975 5500 50  0000 L CNN
+F 1 "47k5" H 3975 5500 50  0000 L CNN
 F 2 "VehicleAccessoryController:R_0603" V 3830 5450 50  0001 C CNN
 F 3 "~" H 3900 5450 50  0001 C CNN
@@
 P 3900 5050
 F 0 "R731" H 3975 5000 50  0000 L CNN
-F 1 "22.1k" H 3975 5100 50  0000 L CNN
+F 1 "22k1" H 3975 5100 50  0000 L CNN
 F 2 "VehicleAccessoryController:R_0603" V 3830 5050 50  0001 C CNN
 F 3 "~" H 3900 5050 50  0001 C CNN

Commit message: correct fuse holder, ACC pull-up, BOM Accessories, create firmware dir
Parts:
- U106: symbol VehicleAccessoryController:Si8621BB-B-IS -> VehicleAccessoryControllerTestBoard-rescue:Si8621BB-B-IS-VehicleAccessoryController
Connections:
- net ACC: no longer R726.2
- net ACC_OUT: now reaches R725.2, U104.6 (VO)
- net ACC_OUT: now also R726.2
Changed lines of the file:
@@
 Sheet 1 1
 Title "Vehicle Accessory Controller Test Board"
-Date "2019-11-22"
+Date "2019-11-29"
 Rev "0.0"
 Comp "Noctivore"
@@
 ACC
 Text Label 1775 5625 2    50   ~ 0
-ACC
+ACC_OUT
 $Comp
 L Device:R R725
@@
 	9275 5150 9425 5150
 $Comp
-L VehicleAccessoryController:Si8621BB-B-IS U106
+L VehicleAccessoryControllerTestBoard-rescue:Si8621BB-B-IS-VehicleAccessoryController U106
 U 1 1 5DC8033B
 P 5550 3675
@@
 	1    0    0    -1
 $EndComp
+Text Label 2700 4150 2    50   ~ 0
+ACC_OUT
 $EndSCHEMATC
