File: hardware/VehicleAccessoryController/VehicleAccessoryController.kicad_pcb (KiCad board)
At the start: 2 copper layers, 242.3 x 146.4 mm, 77 parts, among them J501 Input, J502 Front Conn, J503 Rear Conn, J504 Left Conn, J505 Right Conn, J506 USB_B_Mini, P601 TC2030-MCP, Q201 BSS138, Q202 BSS138, Q203 BSS138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

Commit message: layout updates
Parts:
- moved R720 27.1 mm to (230.5, 90.4), turned to 90 degrees
- moved R723 22.3 mm to (230.5, 121.9), turned to 90 degrees
- moved R719 21.9 mm to (230.5, 118.5), turned to 270 degrees
- moved R717 20.4 mm to (230.5, 97.5), turned to 270 degrees
- moved R721 20.3 mm to (230.5, 100.9), turned to 90 degrees
- moved R712 19.4 mm to (223.5, 90.4), turned to 90 degrees
- moved R718 19.0 mm to (230.5, 108.0), turned to 270 degrees
- moved R716 17.2 mm to (230.5, 87.0), turned to 270 degrees
- moved R708 16.6 mm to (223.5, 87.0), turned to 270 degrees
- moved Q201 15.5 mm to (227.0, 88.7)
- moved J502 15.4 mm to (235.9, 88.7)
- moved R713 13.2 mm to (223.5, 100.9), turned to 90 degrees
- moved R715 12.7 mm to (223.5, 121.9), turned to 90 degrees
- moved R711 12.6 mm to (223.5, 118.5), turned to 270 degrees
- moved R710 12.1 mm to (223.5, 108.0), turned to 270 degrees
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Routing:
- net Net-(J505-Pad2): track 0.00 -> 7.69 mm
- net Net-(J504-Pad2): track 0.00 -> 7.69 mm
- net Net-(J503-Pad2): track 0.00 -> 7.69 mm
- net Net-(J502-Pad2): track 0.00 -> 7.69 mm
- net Net-(Q204-Pad1): track 0.00 -> 4.40 mm
- net Net-(Q203-Pad1): track 0.00 -> 4.40 mm
- net Net-(Q202-Pad1): track 0.00 -> 4.40 mm
- net Net-(Q201-Pad1): track 0.00 -> 4.40 mm
- net Net-(Q204-Pad3): track 0.00 -> 3.92 mm
- net Net-(Q203-Pad3): track 0.00 -> 3.92 mm
- net Net-(Q202-Pad3): track 0.00 -> 3.92 mm
- net Net-(Q201-Pad3): track 0.00 -> 3.92 mm
Other:
- board size 242.3 x 146.4 mm -> 238.9 x 146.4 mm
- board text added: "*"
- board text added: "+"
- board text added: "-"
- board text added: "FRONT"
- board text added: "LEFT"
- board text added: "REAR"
- board text added: "RIGHT"

Commit message: layout updates
Parts:
- added H1: Mounting_Hole, VehicleAccessoryController:Mounting_Hole, F.Cu at (118.8, 70.2)
- added H2: Mounting_Hole, VehicleAccessoryController:Mounting_Hole, F.Cu at (120.5, 136.9)
- moved D603 117.0 mm to (133.3, 133.5), turned to 180 degrees
- moved D604 111.0 mm to (133.0, 130.4), turned to 180 degrees
- moved R729 110.8 mm to (137.3, 133.5), turned to 180 degrees
- moved R730 103.8 mm to (137.1, 130.4), turned to 180 degrees
- moved J501 99.5 mm to (116.6, 83.5)
- moved R701 98.7 mm to (172.4, 93.5), turned to 270 degrees
- moved fid1 96.5 mm to (130.9, 62.8)
- moved F401 88.9 mm to (131.0, 75.4)
- moved fid2 88.4 mm to (132.6, 142.1)
- moved SW301 88.3 mm to (126.3, 115.5)
- moved C801 85.0 mm to (131.0, 88.7), turned to 180 degrees
- moved C804 84.4 mm to (119.0, 97.2)
- moved R703 84.4 mm to (123.7, 100.9)
- moved U103 84.4 mm to (118.7, 103.4)
- moved R704 84.4 mm to (124.1, 97.4)
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Other:
- board size 238.9 x 146.4 mm -> 69.9 x 82.7 mm

Commit message: layout updates
Parts:
- moved fid3 18.3 mm to (156.2, 139.1)
- moved fid1 8.77 mm to (132.0, 71.5)
- moved R724 4.70 mm to (118.4, 123.8)
- moved fid2 3.85 mm to (132.0, 138.3)
- moved R705 3.52 mm to (126.8, 74.6)
- moved H1 3.01 mm to (121.8, 70.5)
- moved C803 2.62 mm to (139.8, 96.9)
- moved U102 2.62 mm to (140.2, 102.3)
- moved C802 2.62 mm to (137.8, 108.1)
- moved P601 2.62 mm to (149.9, 103.1)
- moved R702 2.62 mm to (135.0, 103.6)
- moved Y901 2.62 mm to (141.6, 108.1)
- moved J501 2.40 mm to (119.0, 83.5)
- moved C804 2.31 mm to (121.2, 97.9)
- moved R703 2.22 mm to (125.9, 101.2)
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Other:
- board size 69.9 x 82.7 mm -> 61.4 x 75.2 mm

Commit message: CAD models update
Parts:
- U103: footprint VehicleAccessoryController:TI DSE (S-PWSON-N6) -> VehicleAccessoryController:TI_DSE_(S-PWSON-N6)

Commit message: layout updates
Parts:
- moved R725 20.1 mm to (133.2, 110.2)
- moved C805 20.1 mm to (130.3, 104.8)
- moved R726 20.1 mm to (133.2, 107.4)
- moved U104 20.1 mm to (127.9, 108.9)
- moved R724 16.9 mm to (122.8, 107.5), turned to 270 degrees
- moved D602 12.6 mm to (138.2, 93.4)
- moved R707 12.6 mm to (141.2, 93.4)
- moved D601 12.6 mm to (134.9, 93.3)
- moved R706 12.6 mm to (131.8, 93.3)
- moved SW301 8.40 mm to (126.1, 122.0)
- moved R704 8.12 mm to (119.2, 101.7), turned to 90 degrees
- moved R727 5.45 mm to (153.0, 136.8), turned to 90 degrees
- moved C814 5.30 mm to (161.7, 94.8)
- moved C815 5.30 mm to (154.7, 94.8)
- moved U107 5.30 mm to (158.2, 94.8)
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Routing:
- net /SHIELD: track 0.00 -> 26.5 mm
- net VBUS: track 0.00 -> 6.58 mm
- net /D+: track 0.00 -> 4.83 mm
- net /D-: track 0.00 -> 2.93 mm, vias 0 -> 1
- net GNDD: track 0.00 -> 2.15 mm, vias 0 -> 7
- net VDD: track 0.00 -> 2.00 mm
- added copper zone on F.Cu, net +12VA
- added copper zone on In1.Cu, net +5V
- added copper zone on F.Cu, net GND
- added copper zone on F.Cu, net GNDA
- added copper zone on F.Cu, net GNDD
- added copper zone on F.Cu, net Net-(C801-Pad1)
Other:
- copper layers 2 -> 4
- net class Default: clearance 0.2 -> 0.254; trace_width 0.25 -> 0.254; via_dia 0.8 -> 0.6858; via_drill 0.4 -> 0.3302
- rule trace_clearance: 0.2 -> 0.254
- board text added: "12V"

Commit message: layout updates
Parts:
- moved R705 27.8 mm to (120.4, 100.4), turned to 0 degrees
- moved R729 25.0 mm to (148.2, 113.4)
- moved R730 20.9 mm to (144.8, 113.5)
- moved R704 7.60 mm to (123.9, 95.7), turned to 180 degrees
- moved R703 6.92 mm to (120.0, 95.7), turned to 180 degrees
- moved D603 4.85 mm to (136.5, 132.1), turned to 270 degrees
- moved C804 4.62 mm to (124.2, 100.4)
- moved D601 4.62 mm to (139.4, 94.2)
- moved D602 4.62 mm to (142.7, 94.3)
- moved R706 4.62 mm to (136.3, 94.2)
- moved R707 4.62 mm to (145.7, 94.3)
- moved U103 3.81 mm to (122.0, 98.0)
- moved R728 3.28 mm to (152.2, 115.5)
- moved C811 3.27 mm to (131.0, 119.0), turned to 270 degrees
- moved R732 2.89 mm to (153.2, 118.6), turned to 90 degrees
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Routing:
- net VDD: track 2.00 -> 15.5 mm
- net +5VD: track 0.00 -> 13.0 mm
- net /D+: track 4.83 -> 17.8 mm, vias 0 -> 2
- net /D-: track 2.93 -> 14.3 mm, vias 1 -> 2
- net /CP2102N_RST: track 0.00 -> 5.07 mm
- net /CP2102N_TXD: track 0.00 -> 4.95 mm
- net /CP2102N_RXD: track 0.00 -> 4.64 mm
- net GNDD: track 2.15 -> 6.52 mm, vias 7 -> 8
- net VBUS: track 6.58 -> 8.60 mm, vias 0 -> 1
- added copper zone on B.Cu, net GNDA
Other:
- net class Default: clearance 0.254 -> 0.2; trace_width 0.254 -> 0.25; via_dia 0.6858 -> 0.8; via_drill 0.3302 -> 0.4
- rule trace_clearance: 0.254 -> 0.2
- board text added: "RX"
- board text added: "TX"
