File: hardware/VehicleAccessoryController/VehicleAccessoryController.kicad_pcb (KiCad board)
At the start: 4 copper layers, 61.4 x 75.2 mm, 79 parts, among them J501 Input, J502 Front Conn, J503 Rear Conn, J504 Left Conn, J505 Right Conn, J506 USB_B_Mini, P601 TC2030-MCP, Q201 BSS138, Q202 BSS138, Q203 BSS138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

Commit message: layout updates
Parts:
- moved C804 14.1 mm to (124.3, 114.5)
- moved R705 14.1 mm to (120.3, 114.5)
- moved U103 14.0 mm to (122.3, 112.0)
- moved R704 13.8 mm to (124.3, 109.5)
- moved R703 13.8 mm to (120.3, 109.5)
- moved R706 11.2 mm to (147.5, 94.0)
- moved D601 11.1 mm to (150.5, 94.0)
- moved C805 6.66 mm to (130.6, 96.0), turned to 90 degrees
- moved R726 5.90 mm to (133.2, 100.0)
- moved R724 5.71 mm to (122.3, 101.6), turned to 270 degrees
- moved U104 5.51 mm to (127.9, 101.6)
- moved R725 5.50 mm to (133.2, 103.2)
- moved C814 5.30 mm to (167.0, 94.7)
- moved C815 5.30 mm to (160.0, 94.7)
- moved U107 5.30 mm to (163.5, 94.7)
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Routing:
- net /CTRL: track 0.00 -> 66.6 mm, vias 0 -> 1
- net GND: track 0.00 -> 49.6 mm, vias 0 -> 8
- net /TRIM: track 0.00 -> 28.3 mm, vias 0 -> 1
- net Net-(D603-Pad1): track 0.00 -> 24.7 mm, vias 0 -> 2
- net Net-(D604-Pad1): track 0.00 -> 24.2 mm, vias 0 -> 2
- net /SHUTDOWN: track 0.00 -> 22.2 mm
- net VBUS: track 8.60 -> 28.8 mm, vias 1 -> 2
- net /ACC_IN: track 0.00 -> 19.6 mm
- net GNDD: track 6.52 -> 25.6 mm, vias 8 -> 10
- net +12VA: track 0.00 -> 18.7 mm, vias 0 -> 5
- net +5V: track 0.00 -> 18.7 mm
- net +5VD: track 13.0 -> 31.6 mm, vias 0 -> 5
- net VDD: track 15.5 -> 27.8 mm, vias 0 -> 7
- net GNDA: track 0.00 -> 8.94 mm, vias 0 -> 4
- net Net-(R728-Pad2): track 0.00 -> 6.84 mm
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- added copper zone on In1.Cu, net +12VA
- added copper zone on In1.Cu, net +5VD
- added copper zone on B.Cu, net GND
- added copper zone on B.Cu, net GNDD
- added copper zone on In1.Cu, net VDD
Other:
- net class Default: via_dia 0.8 -> 0.6858; via_drill 0.4 -> 0.3302

Commit message: layout and cad updates
Parts:
- moved P601 1.41 mm to (152.0, 102.6)
- moved C803 1.00 mm to (141.0, 98.0)
- moved C805 1.00 mm to (130.6, 97.0)
- moved R702 1.00 mm to (136.5, 102.6)
- moved R724 1.00 mm to (122.3, 102.6)
- moved R725 1.00 mm to (133.2, 104.2)
- moved R726 1.00 mm to (133.2, 101.0)
- moved U102 1.00 mm to (141.0, 102.6)
- moved U104 1.00 mm to (127.9, 102.6)
- moved Y901 0.71 mm to (143.0, 107.5)
- moved C802 0.66 mm to (139.0, 107.5)
Routing:
- net /328P_MOSI: track 0.00 -> 15.1 mm
- net GND: track 49.6 -> 64.4 mm, vias 8 -> 14
- net /328P_MISO: track 0.00 -> 10.0 mm
- net /328P_SCK: track 0.00 -> 9.59 mm
- net +5VD: track 31.6 -> 40.4 mm, vias 5 -> 7
- net Net-(U102-Pad8): track 0.00 -> 3.50 mm
- net /328P_RST: track 0.00 -> 2.95 mm
- net Net-(U102-Pad7): track 0.00 -> 2.74 mm
- net Net-(C803-Pad1): track 0.00 -> 2.56 mm
- net /POWER_STATUS: track 0.00 -> 1.50 mm, vias 0 -> 1
- net /PARK_STATUS: track 0.00 -> 1.50 mm, vias 0 -> 1
- net /ACC_IN: track 19.6 -> 20.6 mm

Commit message: layout and cad updates, add schematic pdf
Parts:
- moved C811 2.97 mm to (130.4, 121.9), turned to 90 degrees
- moved R702 1.89 mm to (135.5, 101.0), turned to 270 degrees
- moved C803 0.30 mm to (141.0, 97.7)
Connections:
- U102 pad 24: /PARK_REAR -> /PARK_RIGHT
- U102 pad 26: /PARK_RIGHT -> /PARK_REAR
Routing:
- net /PARK_RIGHT: track 1.40 -> 62.8 mm, vias 1 -> 2
- net /328P_RST: track 2.95 -> 62.8 mm, vias 0 -> 5
- net /PARK_LEFT: track 1.40 -> 47.1 mm, vias 1 -> 2
- net /PARK_FRONT: track 1.40 -> 29.7 mm, vias 1 -> 2
- net /PARK_REAR: track 1.40 -> 29.2 mm, vias 1 -> 2
- net /328P_RXD: track 0.00 -> 21.2 mm
- net /328P_TXD: track 0.00 -> 19.0 mm
- net GND: track 64.4 -> 72.1 mm, vias 14 -> 18
- net /ACC: track 0.00 -> 7.53 mm, vias 0 -> 2
- net +5VD: track 40.4 -> 46.7 mm, vias 7 -> 10
- net GNDA: track 8.94 -> 14.4 mm, vias 4 -> 5
- net Net-(C811-Pad2): track 0.00 -> 4.12 mm
- net GNDD: track 25.6 -> 27.0 mm, vias 10 -> 11

Commit message: layout and cad updates
Parts:
- added REF**: Designed_By, VehicleAccessoryController:Designed_By, F.Cu at (164.8, 78.1)
- added REF**: Designed_By, VehicleAccessoryController:Designed_By, F.Cu at (164.0, 77.7)
- moved D601 1.00 mm to (151.5, 94.0)
- moved D602 1.00 mm to (140.5, 94.0)
- moved R706 1.00 mm to (148.5, 94.0)
- moved R707 1.00 mm to (143.5, 94.0)
Routing:
- added copper zone on In2.Cu, net GND
- added copper zone on In2.Cu, net GNDA
- added copper zone on In2.Cu, net GNDD
Other:
- board text added: "Designed by OPS"
- board text added: "PARK"
- board text added: "PWR"

Commit message: layout and firmware updates
Parts:
- moved D601 1.28 mm to (150.5, 93.2)
- moved D602 1.28 mm to (141.5, 93.2)
- moved R706 1.28 mm to (147.5, 93.2)
- moved R707 1.28 mm to (144.5, 93.2)
Connections:
- U102 pad 10: /PARK_STATUS -> (no net)
- U102 pad 19: (no net) -> /PARK_STATUS
- U102 pad 22: (no net) -> /POWER_STATUS
- U102 pad 9: /POWER_STATUS -> (no net)
Routing:
- net GNDA: track 14.4 -> 22.9 mm, vias 5 -> 9
- net Net-(C801-Pad1): track 0.00 -> 6.32 mm
- net GND: track 71.7 -> 76.4 mm, vias 18 -> 20
- net +5V: track 18.7 -> 22.9 mm, vias 0 -> 2
- net +12VA: track 18.7 -> 21.9 mm, vias 5 -> 7
- added copper zone on In1.Cu, net GND
Other:
- board text added: "Vehicle Accessory Controller"
- board text added: "v0.1"

Commit message: schematic/layout updates
Connections:
- U102 pad 19: /PARK_STATUS -> (no net)
- U102 pad 22: /POWER_STATUS -> /PARK_STATUS
- U102 pad 27: Net-(U102-Pad27) -> /POWER_STATUS
- U102 pad 28: Net-(U102-Pad28) -> (no net)
Routing:
- net /POWER_STATUS: track 1.50 -> 22.6 mm, vias 1 -> 2
- net /328P_RST: track 62.8 -> 64.1 mm
- net /PARK_FRONT: track 29.7 -> 28.7 mm
- net GND: track 76.4 -> 75.8 mm

Commit message: schematic/layout updates
Parts:
- turned D601 to 180 degrees
- turned D602 to 0 degrees
Connections:
- D601 pad 1: Net-(D601-Pad1) -> GND
- D601 pad 2: +5VD -> Net-(D601-Pad2)
- D602 pad 1: Net-(D602-Pad1) -> GND
- D602 pad 2: +5VD -> Net-(D602-Pad2)
- R706 pad 1: /PARK_STATUS -> /328P_SCK
- R706 pad 2: Net-(D601-Pad1) -> Net-(D601-Pad2)
- R707 pad 1: /POWER_STATUS -> /PARK_STATUS
- R707 pad 2: Net-(D602-Pad1) -> Net-(D602-Pad2)
- U102 pad 13: Net-(U102-Pad13) -> (no net)
- U102 pad 14: Net-(U102-Pad14) -> (no net)
- U102 pad 22: /PARK_STATUS -> (no net)
- U102 pad 27: /POWER_STATUS -> /PARK_STATUS
Routing:
- net /POWER_STATUS: track 22.6 -> 0.00 mm, vias 2 -> 0
- net /PARK_STATUS: track 1.50 -> 22.6 mm, vias 1 -> 2
- net GND: track 75.8 -> 85.7 mm, vias 20 -> 22
- net /328P_SCK: track 9.59 -> 16.6 mm
- net +5VD: track 46.5 -> 44.0 mm, vias 10 -> 8
- net Net-(D602-Pad2): track 0.00 -> 1.50 mm
- net Net-(D602-Pad1): track 1.50 -> 0.00 mm
- net Net-(D601-Pad2): track 0.00 -> 1.50 mm
- net Net-(D601-Pad1): track 1.50 -> 0.00 mm
Other:
- board text added: "v1.0"
- board text removed: "v0.1"

Commit message: layout updates, gerbers
Routing:
- net GNDD: vias 11 -> 12
Changed lines of the file:
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@@
     (thickness 1.6)
     (drawings 68)
-    (tracks 511)
+    (tracks 512)
     (zones 0)
     (modules 81)
@@
   (title_block
     (title "Vehicle Accessory Controller")
-    (date 2020-06-24)
+    (date 2020-06-26)
     (rev 1.0)
     (company Noctivore)
@@
     (visible_elements FFFFFF7F)
     (pcbplotparams
-      (layerselection 0x010fc_ffffffff)
-      (usegerberextensions false)
+      (layerselection 0x010f8_ffffffff)
+      (usegerberextensions true)
       (usegerberattributes false)
       (usegerberadvancedattributes false)
@@
       (psa4output false)
       (plotreference true)
-      (plotvalue true)
+      (plotvalue false)
       (plotinvisibletext false)
       (padsonsilk false)
@@
       (outputformat 1)
       (mirror false)
-      (drillshape 1)
+      (drillshape 0)
       (scaleselection 1)
-      (outputdirectory ""))
+      (outputdirectory "gerbers/"))
   )
   (net 0 "")
@@
     (add_net VDD)
   )
+  (module "VehicleAccessoryController:TI_DSE_(S-PWSON-N6)" (layer F.Cu)
+    (at 122.3 112)
+    (fp_text reference U103 (at -3.05 0) (layer F.SilkS)
+      (effects (font (size 1 1) (thickness 0.15)))
+    )
+    (fp_text value TPS3710 (at 1.2 0 90) (layer F.Fab)
+      (effects (font (size 0.3 0.3) (thickness 0.075) italic))
+    )
+    (fp_line (start -0.75 -0.75) (end 0.75 -0.75) (layer F.SilkS) (width 0.15))
+    (fp_line (start 0.75 -0.75) (end 0.75 0.75) (layer F.SilkS) (width 0.15))
+    (fp_line (start 0.75 0.75) (end -0.75 0.75) (layer F.SilkS) (width 0.15))
+    (fp_line (start -0.75 0.75) (end -0.75 -0.75) (layer F.SilkS) (width 0.15))
+    (fp_circle (center -0.5 1.2) (end -0.4 1.2) (layer F.SilkS) (width 0.15))
+    (pad 1 smd custom (at -0.5 0.525) (size 0.1 0.1) (layers F.Cu F.Paste F.Mask)
+      (net 2 GNDA) (solder_mask_margin 0.05) (solder_paste_margin -0.01) (clearance 0.05) (zone_connect 0)
+      (options (clearance outline) (anchor rect))
+      (primitives
+        (gr_poly (pts
+           (xy -0.14 0.425) (xy 0.14 0.425) (xy 0.14 -0.425) (xy 0 -0.425) (xy -0.14 -0.285)
+) (width 0))
+      ))
+    (pad 3 smd rect (at 0.5 0.575) (size 0.28 0.75) (layers F.Cu F.Paste F.Mask)
+      (net 2 GNDA) (solder_mask_margin 0.05) (solder_paste_margin -0.01) (clearance 0.05))
+    (pad 2 smd rect (at 0 0.575) (size 0.28 0.75) (layers F.Cu F.Paste F.Mask)
+      (net 6 +12VA) (solder_mask_margin 0.05) (solder_paste_margin -0.01) (clearance 0.05))
+    (pad 4 smd rect (at 0.5 -0.575) (size 0.28 0.75) (layers F.Cu F.Paste F.Mask)
+      (net 34 "Net-(R703-Pad1)") (solder_mask_margin 0.05) (solder_paste_margin -0.01) (clearance 0.05))
+    (pad 5 smd rect (at 0 -0.575) (size 0.28 0.75) (layers F.Cu F.Paste F.Mask)
+      (net 2 GNDA) (solder_mask_margin 0.05) (solder_paste_margin -0.01) (clearance 0.05))
+    (pad 6 smd rect (at -0.5 -0.575) (size 0.28 0.75) (layers F.Cu F.Paste F.Mask)
+      (net 47 /SHUTDOWN) (solder_mask_margin 0.05) (solder_paste_margin -0.01) (clearance 0.05))
+    (model ${KISYS3DMOD}/Package_SON.3dshapes/WSON-6_1.5x1.5mm_P0.5mm.step
+      (at (xyz 0 0 0))
+      (scale (xyz 1 1 1))
+      (rotate (xyz 0 0 0))
+    )
+  )
   (module VehicleAccessoryController:REM20-XXXXXW (layer F.Cu)
     (at 157.9 78.2)
@@
     )
   )
-  (module "VehicleAccessoryController:TI_DSE_(S-PWSON-N6)" (layer F.Cu)
-    (at 122.3 112)
-    (fp_text reference U103 (at -3.05 0) (layer F.SilkS)
-      (effects (font (size 1 1) (thickness 0.15)))
-    )
-    (fp_text value TPS3710 (at -1.14 0.06 90) (layer F.Fab)
-      (effects (font (size 0.3 0.3) (thickness 0.075)))
-    )
-    (fp_line (start -0.75 -0.75) (end 0.75 -0.75) (layer F.SilkS) (width 0.15))
-    (fp_line (start 0.75 -0.75) (end 0.75 0.75) (layer F.SilkS) (width 0.15))
-    (fp_line (start 0.75 0.75) (end -0.75 0.75) (layer F.SilkS) (width 0.15))
-    (fp_line (start -0.75 0.75) (end -0.75 -0.75) (layer F.SilkS) (width 0.15))
-    (pad 1 smd custom (at -0.5 0.525) (size 0.1 0.1) (layers F.Cu F.Paste F.Mask)
-      (net 2 GNDA) (solder_mask_margin 0.05) (solder_paste_margin -0.01) (clearance 0.05) (zone_connect 0)
-      (options (clearance outline) (anchor rect))
-      (primitives
-        (gr_poly (pts
-           (xy -0.14 0.425) (xy 0.14 0.425) (xy 0.14 -0.425) (xy 0 -0.425) (xy -0.14 -0.285)
-) (width 0))
-      ))
-    (pad 3 smd rect (at 0.5 0.575) (size 0.28 0.75) (layers F.Cu F.Paste F.Mask)
-      (net 2 GNDA) (solder_mask_margin 0.05) (solder_paste_margin -0.01) (clearance 0.05))
-    (pad 2 smd rect (at 0 0.575) (size 0.28 0.75) (layers F.Cu F.Paste F.Mask)
-      (net 6 +12VA) (solder_mask_margin 0.05) (solder_paste_margin -0.01) (clearance 0.05))
-    (pad 4 smd rect (at 0.5 -0.575) (size 0.28 0.75) (layers F.Cu F.Paste F.Mask)
-      (net 34 "Net-(R703-Pad1)") (solder_mask_margin 0.05) (solder_paste_margin -0.01) (clearance 0.05))
-    (pad 5 smd rect (at 0 -0.575) (size 0.28 0.75) (layers F.Cu F.Paste F.Mask)
-      (net 2 GNDA) (solder_mask_margin 0.05) (solder_paste_margin -0.01) (clearance 0.05))
-    (pad 6 smd rect (at -0.5 -0.575) (size 0.28 0.75) (layers F.Cu F.Paste F.Mask)
-      (net 47 /SHUTDOWN) (solder_mask_margin 0.05) (solder_paste_margin -0.01) (clearance 0.05))
-    (model ${KISYS3DMOD}/Package_SON.3dshapes/WSON-6_1.5x1.5mm_P0.5mm.step
-      (at (xyz 0 0 0))
-      (scale (xyz 1 1 1))
-      (rotate (xyz 0 0 0))
-    )
-  )
   (module VehicleAccessoryController:Keystone_8719 (layer F.Cu)
     (at 119 83.5 270)
@@
       (effects (font (size 1 1) (thickness 0.15)) (justify mirror))
     )
-    (fp_text value USB_B_Mini (at 0 5.1) (layer F.Fab)
+    (fp_text value USB_B_Mini (at 0 5.08) (layer F.Fab)
       (effects (font (size 0.7 0.7) (thickness 0.15)))
     )
@@
   (via (at 139.475 113.4) (size 0.6858) (drill 0.3302) (layers F.Cu B.Cu) (net 8))
   (segment (start 139.475 114.555) (end 139.475 113.4) (width 0.254) (layer F.Cu) (net 8))
+  (via (at 146 119) (size 0.6858) (drill 0.3302) (layers F.Cu B.Cu) (net 8))
   (segment (start 151.1 126) (end 151.1 128) (width 0.508) (layer F.Cu) (net 9))
   (segment (start 146.75 120.9375) (end 147.25 120.9375) (width 0.25) (layer F.Cu) (net 9))
@@
   (segment (start 133.3 132.85) (end 131.8 132.85) (width 0.254) (layer F.Cu) (net 9))
   (via (at 138.475 127.45) (size 0.6858) (drill 0.3302) (layers F.Cu B.Cu) (net 9))
-  (via (at 141.5 115.825) (size 0.6858) (drill 0.3302) (layers F.Cu B.Cu) (net 9))
-  (segment (start 139.475 115.825) (end 141.5 115.825) (width 0.254) (layer F.Cu) (net 9))
+  (via (at 141.3 115.825) (size 0.6858) (drill 0.3302) (layers F.Cu B.Cu) (net 9))
   (segment (start 138.475 125.5) (end 138.475 127.45) (width 0.254) (layer F.Cu) (net 9))
   (via (at 154.5 114.6) (size 0.6858) (drill 0.3302) (layers F.Cu B.Cu) (net 9))
   (segment (start 152.85 114.6) (end 154.5 114.6) (width 0.254) (layer F.Cu) (net 9))
+  (segment (start 139.475 115.825) (end 141.3 115.825) (width 0.254) (layer F.Cu) (net 9))
   (segment (start 153 133.82) (end 151.75 133.82) (width 0.254) (layer F.Cu) (net 10))
   (segment (start 150.45 132.52) (end 150.45 132.27) (width 0.254) (layer F.Cu) (net 10))
