File: hardware/VehicleAccessoryController/VehicleAccessoryController.sch (KiCad schematic (older format))
At the start: 78 parts, among them J501 Input, J502 Front Conn, J503 Rear Conn, J504 Left Conn, J505 Right Conn, J506 USB_B_Mini, P601 TC2030-MCP, Q201 BSS138, Q202 BSS138, Q203 BSS138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

Commit message: layout and cad updates, add schematic pdf
Changed lines of the file:
@@
 Sheet 1 1
 Title "Vehicle Accessory Controller"
-Date "2019-12-03"
+Date "2020-06-22"
 Rev "0.1"
 Comp "Noctivore"
@@
 Text Label 6525 2775 0    50   ~ 0
 PARK_FRONT
-Text Label 6525 2875 0    50   ~ 0
+Text Label 6525 3075 0    50   ~ 0
 PARK_REAR
 Text Label 6525 2975 0    50   ~ 0
 PARK_LEFT
-Text Label 6525 3075 0    50   ~ 0
+Text Label 6525 2875 0    50   ~ 0
 PARK_RIGHT
 Text Label 4825 2275 2    50   ~ 0

Commit message: schematic/layout updates
Connections:
- no-connect marks 14 -> 12
Changed lines of the file:
@@
 Sheet 1 1
 Title "Vehicle Accessory Controller"
-Date "2020-06-23"
+Date "2020-06-24"
 Rev "0.1"
 Comp "Noctivore"
@@
 Wire Wire Line
 	4225 1675 4225 1575
-NoConn ~ 4975 2375
-NoConn ~ 4975 2475
 NoConn ~ 6375 2475
 $Comp

Commit message: schematic/layout updates
Parts:
- U103: footprint VehicleAccessoryController:TI DSE (S-PWSON-N6) -> VehicleAccessoryController:TI_DSE_(S-PWSON-N6)
Connections:
- net labels removed: POWER_STATUS
- wire segments 267 -> 266
- no-connect marks 12 -> 10
Other:
- note added: "(POWER_STATUS)"
- moved on the sheet: C802, C803, D601, D602, P601, R702, U102, Y901
